Commit message: scout raw

File: scout2/urdf/scout2.urdf (robot description, URDF)
Before this commit: robot scout2, 1 links, 0 joints
Links:
- added link base_footprint
- added link camholder_1; visual box size=0.1 0.04 0.005
- added link camholder_2; visual box size=0.01 0.04 0.04
- added link caster_wheel; visual sphere radius=0.015
- added link chassis_casterWheel_cylinder; visual cylinder length=0.09 radius=0.015
- added link chassis_front_cylinder; visual cylinder length=0.025 radius=0.06
- added link chassis_lidar_block; visual box size=0.03 0.105 0.05
- added link chassis_main; visual box size=0.32 0.105 0.07
- added link chassis_main_top; visual box size=0.22 0.105 0.05
- added link chassis_tail_cylinder; visual cylinder length=0.12 radius=0.0525
- added link lidar; visual cylinder length=0.03 radius=0.05
- added link wheel_deko_left; visual cylinder length=0.001 radius=0.025
- added link wheel_deko_right; visual cylinder length=0.001 radius=0.025
- added link wheel_holder_left; visual cylinder length=0.1 radius=0.03
- added link wheel_holder_right; visual cylinder length=0.1 radius=0.03
- added link wheel_left; visual cylinder length=0.045 radius=0.0625
- added link wheel_right; visual cylinder length=0.045 radius=0.0625
- link base_link: geometry visual box size=0.025 0.15 0.02
Joints:
- added joint base_footprint: type fixed, parent base_footprint, child base_link, origin xyz=0.0 0.0 0.085 rpy=0.0 0.0 0.0
- added joint camholder_main: type fixed, parent camholder_1, child camholder_2, origin xyz=0.04 0.0 0.0 rpy=0.0 0.0 0.0
- added joint casterWheel: type fixed, parent chassis_casterWheel_cylinder, child caster_wheel, origin xyz=0 0 -0.09 rpy=0.0 0.0 0.0
- added joint chassi_1: type fixed, parent base_link, child wheel_holder_right, origin xyz=0.0 -0.035 -0.02 rpy=0.0 0.0 0.0
- added joint chassi_2: type fixed, parent base_link, child wheel_holder_left, origin xyz=0.0 0.035 -0.02 rpy=0.0 0.0 0.0
- added joint chassi_base: type fixed, parent base_link, child chassis_main, origin xyz=-0.08 0.0 0.02 rpy=0.0 0.0 0.0
- added joint chassi_base_cylinder: type fixed, parent chassis_main, child chassis_tail_cylinder, origin xyz=-0.16 0 0 rpy=0.0 0.0 0.0
- added joint chassi_base_top: type fixed, parent chassis_main, child chassis_main_top, origin xyz=-0.05 0.0 0.07 rpy=0.0 0.0 0.0
- added joint chassi_casterWheel_cylinder: type fixed, parent chassis_tail_cylinder, child chassis_casterWheel_cylinder, origin xyz=0 0 0 rpy=0.0 0.0 0.0
- added joint chassi_front_cylinder: type fixed, parent chassis_main, child chassis_front_cylinder, origin xyz=0.135 0 0.07 rpy=0.0 0.0 0.0
- added joint chassis_lidar: type fixed, parent chassis_main, child chassis_lidar_block, origin xyz=0.045 0.0 0.12 rpy=0.0 0.0 0.0
- added joint deko_1: type fixed, parent wheel_right, child wheel_deko_right, origin xyz=0.0 -0.045 0 rpy=0.0 0.0 0.0
- added joint deko_2: type fixed, parent wheel_left, child wheel_deko_left, origin xyz=0.0 0.045 0 rpy=0.0 0.0 0.0
- added joint joint_1: type revolute, parent wheel_holder_right, child wheel_right, origin xyz=0 -0.1 0 rpy=0 0 0, axis 0 1 0, limit lower=-3.14159 upper=3.14159 effort=1000.0 velocity=50.0
- added joint joint_2: type revolute, parent wheel_holder_left, child wheel_left, origin xyz=0 0.1 0 rpy=0 0 0, axis 0 1 0, limit lower=-3.14159 upper=3.14159 effort=1000.0 velocity=50.0
- added joint mount_lidar: type fixed, parent chassis_lidar_block, child lidar, origin xyz=0.0 0.0 0.05 rpy=0.0 0.0 0.0
- added joint move_cam_joint: type fixed, parent chassis_front_cylinder, child camholder_1, origin xyz=0.0 0.0 0.02 rpy=0.0 0.0 0.0
