Commit message: added Gazebo Colors

File: scout2/urdf/camera.xacro (robot description, xacro)
@@ -19,4 +19,7 @@
                            xyz="0.0 0.0 0.0015" rpy="0 0 0"/>
     </link>
+    <gazebo reference="camholder_1">
+        <material>Gazebo/Black</material>
+    </gazebo>
     <link name="camholder_2">
         <visual>
@@ -36,4 +39,7 @@
                            xyz="0.0 0.0 0.02" rpy="0 0 0"/>
     </link>
+    <gazebo reference="camholder_2">
+        <material>Gazebo/Black</material>
+    </gazebo>
     <!-- Joint now Fixed but later Moving -->
     <joint name="move_cam_joint" type="fixed">

File: scout2/urdf/lidar.xacro (robot description, xacro)
@@ -19,4 +19,7 @@
             xyz="0.0 0.0 0.025" rpy="0 0 0" />
     </link>
+    <gazebo reference="chassis_lidar_block">
+        <material>Gazebo/Black</material>
+    </gazebo>
     <link name="lidar">
         <visual>
@@ -36,4 +39,7 @@
                            xyz="0.0 0.0 0.015" rpy="0 0 0"/>
     </link>
+    <gazebo reference="lidar">
+        <material>Gazebo/Red</material>
+    </gazebo>
     <joint name="chassis_lidar" type="fixed">
         <parent link="chassis_main" />

File: scout2/urdf/rover.xacro (robot description, xacro)
@@ -20,4 +20,7 @@
             xyz="0.0 0.0 0.01" rpy="0 0 0" />
     </link>
+    <gazebo reference="base_link">
+        <material>Gazebo/Black</material>
+    </gazebo>
     <!--  WHEELS AND DEKO -->
     <xacro:macro name="wh_link" params="prefix y">
@@ -39,4 +42,7 @@
                 xyz="0 ${y} 0" rpy="0 0 0" />
         </link>
+        <gazebo reference="wheel_holder_${prefix}">
+            <material>Gazebo/Black</material>
+        </gazebo>
     </xacro:macro>
     <xacro:wh_link prefix="right" y="-0.05" />
@@ -60,4 +66,7 @@
                 xyz="0 ${y} 0" rpy="0 0 0" />
         </link>
+        <gazebo reference="wheel_${prefix}">
+            <material>Gazebo/Black</material>
+        </gazebo>
     </xacro:macro>
     <xacro:wheel_link prefix="right" y="-0.0225" />
@@ -81,4 +90,7 @@
                 xyz="0 0 0" rpy="1.57 0.0 0.0" />
         </link>
+        <gazebo reference="wheel_deko_${prefix}">
+            <material>Gazebo/White</material>
+        </gazebo>
     </xacro:macro>
     <xacro:wheel_deko prefix="right" />
@@ -102,4 +114,7 @@
             xyz="0.0 0.0 0.035" rpy="0 0 0" />
     </link>
+    <gazebo reference="chassis_main">
+        <material>Gazebo/Orange</material>
+    </gazebo>
     <link name="chassis_main_top">
         <visual>
@@ -119,4 +134,7 @@
             xyz="0.0 0.0 0.025" rpy="0 0 0" />
     </link>
+    <gazebo reference="chassis_main_top">
+        <material>Gazebo/Orange</material>
+    </gazebo>
     <link name="chassis_tail_cylinder">
         <visual>
@@ -136,4 +154,7 @@
             xyz="0.0 0.0 0.06" rpy="0 0 0" />
     </link>
+    <gazebo reference="chassis_tail_cylinder">
+        <material>Gazebo/Orange</material>
+    </gazebo>
     <link name="chassis_front_cylinder">
         <visual>
@@ -153,4 +174,7 @@
             xyz="0.0 0.0 -0.0125" rpy="0 0 0" />
     </link>
+    <gazebo reference="chassis_front_cylinder">
+        <material>Gazebo/Orange</material>
+    </gazebo>
     <link name="chassis_casterWheel_cylinder">
         <visual>
@@ -170,4 +194,7 @@
             xyz="0.0 0.0 -0.045" rpy="0 0 0" />
     </link>
+    <gazebo reference="chassis_casterWheel_cylinder">
+        <material>Gazebo/Orange</material>
+    </gazebo>
     <link name="caster_wheel">
         <visual>
@@ -187,3 +214,6 @@
             xyz="0 0 0" rpy="0 0 0" />
     </link>
+    <gazebo reference="caster_wheel">
+        <material>Gazebo/Black</material>
+    </gazebo>
 </robot>
