Commit message: lidar in gz works

File: scout2/urdf/lidar.xacro (robot description, xacro)
@@ -64,5 +64,5 @@
                 </ros>
                 <output_type>sensor_msgs/LaserScan</output_type>
-                <frame_name>laser_frame</frame_name>
+                <frame_name>lidar</frame_name>
             </plugin>
         </sensor>
@@ -76,5 +76,5 @@
         <parent link="chassis_lidar_block" />
         <child link="lidar" />
-        <origin xyz="0.0 0.0 0.05" rpy="0.0 0.0 0.0" />
+        <origin xyz="0.0 0.0 0.05" rpy="0.0 0.0 ${-pi/2}" />
     </joint>
 </robot>
