Commit message: scout ueberschlaegt sich

File: scout2/urdf/joints.xacro (robot description, xacro)
@@ -61,16 +61,16 @@
     <!-- Moving Joints -->
     <joint name="joint_1" type="revolute">
-        <parent link="wheel_holder_right" />
+        <parent link="base_link" />
         <child link="wheel_right" />
         <axis xyz="0 1 0" />
         <limit lower="-3.14159" upper="3.14159" velocity="50.0" effort="1000.0" />
-        <origin xyz="0 -0.1 0" rpy="0 0 0" />
+        <origin xyz="0 -0.135 -0.02" rpy="0 0 0" />
     </joint>
     <joint name="joint_2" type="revolute">
-        <parent link="wheel_holder_left" />
+        <parent link="base_link" />
         <child link="wheel_left" />
         <axis xyz="0 1 0" />
         <limit lower="-3.14159" upper="3.14159" velocity="50.0" effort="1000.0" />
-        <origin xyz="0 0.1 0" rpy="0 0 0" />
+        <origin xyz="0 0.135 -0.02" rpy="0 0 0" />
     </joint>
 </robot>

File: scout2/urdf/rover.xacro (robot description, xacro)
@@ -17,5 +17,5 @@
             </geometry>
         </collision>
-        <xacro:box_inertia m="0.5" l="0.025" w="0.15" h="0.02"
+        <xacro:box_inertia m="0.2" l="0.025" w="0.15" h="0.02"
             xyz="0.0 0.0 0.01" rpy="0 0 0" />
     </link>
@@ -193,5 +193,5 @@
             </geometry>
         </collision>
-        <xacro:cylinder_inertia m="0.05" r="0.015" h="0.09"
+        <xacro:cylinder_inertia m="0.3" r="0.015" h="0.09"
             xyz="0.0 0.0 -0.045" rpy="0 0 0" />
     </link>
@@ -213,5 +213,5 @@
             </geometry>
         </collision>
-        <xacro:sphere_inertia m="0.1" r="0.015"
+        <xacro:sphere_inertia m="0.05" r="0.015"
             xyz="0 0 0" rpy="0 0 0" />
     </link>

Commit message: joint war falsch gewählt

File: scout2/urdf/joints.xacro (robot description, xacro)
@@ -60,17 +60,15 @@
     </joint>
     <!-- Moving Joints -->
-    <joint name="joint_1" type="revolute">
+    <joint name="joint_1" type="continuous">
         <parent link="base_link" />
         <child link="wheel_right" />
         <axis xyz="0 1 0" />
-        <limit lower="-3.14159" upper="3.14159" velocity="50.0" effort="1000.0" />
-        <origin xyz="0 -0.135 -0.02" rpy="0 0 0" />
+        <origin xyz="0 -0.136 -0.02" rpy="0 0 0" />
     </joint>
-    <joint name="joint_2" type="revolute">
+    <joint name="joint_2" type="continuous">
         <parent link="base_link" />
         <child link="wheel_left" />
         <axis xyz="0 1 0" />
-        <limit lower="-3.14159" upper="3.14159" velocity="50.0" effort="1000.0" />
-        <origin xyz="0 0.135 -0.02" rpy="0 0 0" />
+        <origin xyz="0 0.136 -0.02" rpy="0 0 0" />
     </joint>
 </robot>

File: scout2/urdf/rover.xacro (robot description, xacro)
@@ -113,5 +113,5 @@
             </geometry>
         </collision>
-        <xacro:box_inertia m="0.5" l="0.32" w="0.105" h="0.07"
+        <xacro:box_inertia m="2.0" l="0.32" w="0.105" h="0.07"
             xyz="0.0 0.0 0.035" rpy="0 0 0" />
     </link>
@@ -133,5 +133,5 @@
             </geometry>
         </collision>
-        <xacro:box_inertia m="0.2" l="0.22" w="0.105" h="0.05"
+        <xacro:box_inertia m="1.0" l="0.22" w="0.105" h="0.05"
             xyz="0.0 0.0 0.025" rpy="0 0 0" />
     </link>
@@ -153,5 +153,5 @@
             </geometry>
         </collision>
-        <xacro:cylinder_inertia m="0.2" r="0.0525" h="0.12"
+        <xacro:cylinder_inertia m="0.4" r="0.0525" h="0.12"
             xyz="0.0 0.0 0.06" rpy="0 0 0" />
     </link>
